Commit message: simple simple works

File: rl-gripper/rl_gripper/resources/models/xarm6_with_gripper_with_camera_effort_bottom.urdf (robot description, URDF)
Before this commit: robot xarm6_with_gripper, 17 links, 16 joints
Joints:
- joint camera_joint: origin xyz=0 0 0.11 rpy=0 0 0 -> xyz=0 0 0.13 rpy=0 0 0
