Commit message: curriculum for workspace

File: rl-gripper/rl_gripper/resources/models/robot.urdf (robot description, URDF)
Before this commit: robot xarm6_with_gripper, 17 links, 16 joints
Links:
- link camera_link: geometry visual box size=0.013 0.013 0.02
- link tcp_link: mass None -> 0.001
Joints:
- joint camera_joint: origin xyz=0 0 0.115 rpy=0 0 0 -> xyz=0 0 0.10 rpy=0 0 0
- joint tcp_joint: origin xyz=0 0 0.15 rpy=0 0 0 -> xyz=0 0 0.16 rpy=0 0 0
