Commit message: Observation now with raw depth pixels! - Rewarding green pixels only

File: rl-gripper/rl_gripper/resources/models/cube.urdf (robot description, URDF)
Before this commit: robot cube.urdf, 1 links, 0 joints
Links:
- link base_cube_link: geometry collision box size=0.05 0.05 0.05; visual box size=0.05 0.05 0.05

File: rl-gripper/rl_gripper/resources/models/xarm6_with_gripper_with_camera_effort.urdf (robot description, URDF)
Before this commit: robot xarm6_with_gripper, 17 links, 16 joints
Joints:
- joint camera_joint: origin xyz=0.08 0 0.05 rpy=0 -0.35 0 -> xyz=0.08 0 0.05 rpy=0 -0.23 0

Commit message: recent

File: rl-gripper/rl_gripper/resources/models/cube.urdf (robot description, URDF)
Before this commit: robot cube.urdf, 1 links, 0 joints
Links:
- link base_cube_link: mass 0.02 -> 0.01; geometry collision box size=0.035 0.035 0.035; visual box size=0.035 0.035 0.035

Commit message: backup

File: rl-gripper/rl_gripper/resources/models/cube.urdf (robot description, URDF)
Before this commit: robot cube.urdf, 1 links, 0 joints
Links:
- link base_cube_link: mass 0.01 -> 0.2

File: rl-gripper/rl_gripper/resources/models/xarm6_with_gripper_with_camera_effort_bottom.urdf (robot description, URDF)
Before this commit: robot xarm6_with_gripper, 17 links, 16 joints
Links:
- link camera_link: geometry visual box size=0.013 0.013 0.05
Joints:
- joint camera_joint: origin xyz=0 0 0.13 rpy=0 0 0 -> xyz=0 0 0.11 rpy=0 0 0

Commit message: backup

File: rl-gripper/rl_gripper/resources/models/cube.urdf (robot description, URDF)
Before this commit: robot cube.urdf, 1 links, 0 joints
Links:
- link base_cube_link: mass 0.2 -> 0.08

File: rl-gripper/rl_gripper/resources/models/xarm6_with_gripper_with_camera_effort_bottom.urdf (robot description, URDF)
Before this commit: robot xarm6_with_gripper, 17 links, 16 joints
Links:
- link camera_link: geometry visual box size=0.013 0.013 0.03
Joints:
- joint camera_joint: origin xyz=0 0 0.11 rpy=0 0 0 -> xyz=0 0 0.115 rpy=0 0 0

Commit message: working with coordinate-based inputs

File: rl-gripper/rl_gripper/resources/models/cube.urdf (robot description, URDF)
Before this commit: robot cube.urdf, 1 links, 0 joints
Links:
- link base_cube_link: mass 0.08 -> 0.1

Commit message: vision based working

File: rl-gripper/rl_gripper/resources/models/cube.urdf (robot description, URDF)
Before this commit: robot cube.urdf, 1 links, 0 joints
Links:
- link base_cube_link: geometry collision box size=0.04 0.04 0.04; visual box size=0.04 0.04 0.04
